File: hardware/kicad/PET_project/PET_project.kicad_sch (KiCad schematic)
At the start: 21 parts, among them J1 Conn_01x02_Socket, J2 Screw_Terminal_01x02, J3 Screw_Terminal_01x02, J4 Conn_01x02_Socket, J5 GY-GPSV2-NEO6M, J6 BMM350, J7 MPU6050, J8 Conn_01x02_Socket, J9 BMP280, Q2 NMOS, Q3 NMOS, U8 LM317_TO-220

Commit message: board
Parts:
- C1: footprint Capacitor_THT:CP_Radial_Tantal_D5.0mm_P2.50mm -> Capacitor_THT:CP_Radial_Tantal_D4.5mm_P5.00mm
- C2: value 0.33 -> 22; footprint Capacitor_THT:CP_Radial_Tantal_D5.0mm_P2.50mm -> Capacitor_THT:C_Radial_D5.0mm_H11.0mm_P2.00mm
- J5: footprint my_footprint:NEO6M_PinSocket_Vertical -> my_footprint:GY-GPSV2-NEO6M
- U8: value LM317_TO-220 -> BA50DD0T
Changed lines of the file:
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@@
 			)
 		)
-		(property "Value" "LM317_TO-220"
+		(property "Value" "BA50DD0T"
 			(at 83.82 26.67 0)
 			(show_name no)
@@
 			)
 		)
-		(property "Value" "0.33"
+		(property "Value" "22"
 			(at 97.79 35.5599 0)
 			(show_name no)
@@
 			)
 		)
-		(property "Footprint" "Capacitor_THT:CP_Radial_Tantal_D5.0mm_P2.50mm"
+		(property "Footprint" "Capacitor_THT:C_Radial_D5.0mm_H11.0mm_P2.00mm"
 			(at 94.9452 38.1 0)
 			(hide yes)
@@
 			)
 		)
-		(property "Footprint" "my_footprint:NEO6M_PinSocket_Vertical"
+		(property "Footprint" "my_footprint:GY-GPSV2-NEO6M"
 			(at 128.27 55.88 0)
 			(hide yes)
@@
 			)
 		)
-		(property "Footprint" "Capacitor_THT:CP_Radial_Tantal_D5.0mm_P2.50mm"
+		(property "Footprint" "Capacitor_THT:CP_Radial_Tantal_D4.5mm_P5.00mm"
 			(at 73.3552 38.1 0)
 			(hide yes)
