File: hardware/kicad/PET_project/PET_project.kicad_pcb (KiCad board)
At the start: 2 copper layers, 110 x 50 mm, 29 parts, among them J10 Conn_01x06_Socket, J2 Screw_Terminal_01x02, J3 Screw_Terminal_01x02, J5 GY-GPSV2-NEO6M, J6 Conn_01x06_Socket, J7 MPU6050, J8 Conn_01x02_Socket, J9 BMP280, Q2 NMOS, Q3 NMOS, U3 MCP23008-xP, U4 BA50DD0T

Commit message: ドライバの穴修正
Routing:
- net Net-(J6-Pin_1): track 27.5 -> 26.4 mm
- net Net-(U2-STBY): track 10.3 -> 10.8 mm
- net Net-(U2-BIN2): track 10.3 -> 10.8 mm
- net Net-(U2-BIN1): track 10.3 -> 10.8 mm
- net Net-(U2-AIN2): track 10.3 -> 10.8 mm
- net Net-(U2-AIN1): track 10.3 -> 10.8 mm
- net Net-(J6-Pin_6): track 42.9 -> 43.4 mm
- net +3V3: track 256.3 -> 256.8 mm
Changed lines of the file:
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@@
 		(sheetname "/")
 		(sheetfile "PET_project.kicad_sch")
-		(units
-			(unit
-				(name "A")
-				(pins "1" "2" "3" "4" "5" "6" "7" "8" "16" "15" "14" "13" "12" "11" "10"
-					"9"
-				)
-			)
-		)
 		(attr through_hole)
 		(duplicate_pad_numbers_are_jumpers no)
 		(fp_rect
-			(start -10.25 -10.2)
-			(end 10.25 10.2)
+			(start -10.25 -10.207628)
+			(end 10.241179 10.2)
 			(stroke
 				(width 0.1)
@@
 		)
 		(pad "1" thru_hole circle
-			(at -8.25 -8.89 270)
+			(at -7.75 -8.89 270)
 			(size 1.8 1.8)
 			(drill 1)
@@
 		)
 		(pad "2" thru_hole circle
-			(at -8.25 -6.35 270)
+			(at -7.75 -6.35 270)
 			(size 1.8 1.8)
 			(drill 1)
@@
 		)
 		(pad "3" thru_hole circle
-			(at -8.25 -3.81 270)
+			(at -7.75 -3.81 270)
 			(size 1.8 1.8)
 			(drill 1)
@@
 		)
 		(pad "4" thru_hole circle
-			(at -8.25 -1.27 270)
+			(at -7.75 -1.27 270)
 			(size 1.8 1.8)
 			(drill 1)
@@
 		)
 		(pad "5" thru_hole circle
-			(at -8.25 1.27 270)
+			(at -7.75 1.27 270)
 			(size 1.8 1.8)
 			(drill 1)
@@
 		)
 		(pad "6" thru_hole circle
-			(at -8.25 3.81 270)
+			(at -7.75 3.81 270)
 			(size 1.8 1.8)
 			(drill 1)
@@
 		)
 		(pad "7" thru_hole circle
-			(at -8.25 6.35 270)
+			(at -7.75 6.35 270)
 			(size 1.8 1.8)
 			(drill 1)
@@
 		)
 		(pad "8" thru_hole circle
-			(at -8.25 8.89 270)
+			(at -7.75 8.89 270)
 			(size 1.8 1.8)
 			(drill 1)
@@
 		)
 		(pad "9" thru_hole circle
-			(at 8.25 8.89 270)
+			(at 7.75 8.89 270)
 			(size 1.8 1.8)
 			(drill 1)
@@
 		)
 		(pad "10" thru_hole circle
-			(at 8.25 6.35 270)
+			(at 7.75 6.35 270)
 			(size 1.8 1.8)
 			(drill 1)
@@
 		)
 		(pad "11" thru_hole circle
-			(at 8.25 3.81 270)
+			(at 7.75 3.81 270)
 			(size 1.8 1.8)
 			(drill 1)
@@
 		)
 		(pad "12" thru_hole circle
-			(at 8.25 1.27 270)
+			(at 7.75 1.27 270)
 			(size 1.8 1.8)
 			(drill 1)
@@
 		)
 		(pad "13" thru_hole circle
-			(at 8.25 -1.27 270)
+			(at 7.75 -1.27 270)
 			(size 1.8 1.8)
 			(drill 1)
@@
 		)
 		(pad "14" thru_hole circle
-			(at 8.25 -3.81 270)
+			(at 7.75 -3.81 270)
 			(size 1.8 1.8)
 			(drill 1)
@@
 		)
 		(pad "15" thru_hole circle
-			(at 8.25 -6.35 270)
+			(at 7.75 -6.35 270)
 			(size 1.8 1.8)
 			(drill 1)
@@
 		)
 		(pad "16" thru_hole circle
-			(at 8.25 -8.89 270)
+			(at 7.75 -8.89 270)
 			(size 1.8 1.8)
 			(drill 1)
@@
 	)
 	(segment
-		(start 134.25 103.75)
-		(end 126.89 103.75)
-		(width 1)
-		(layer "F.Cu")
-		(net "+6V")
-	)
-	(segment
 		(start 160 110.5)
 		(end 155.5 115)
@@
 	)
 	(segment
-		(start 138.5 108)
-		(end 134.25 103.75)
-		(width 1)
-		(layer "F.Cu")
-		(net "+6V")
-	)
-	(segment
 		(start 142.5 110.5)
 		(end 142.5 125.5)
@@
 	)
 	(segment
+		(start 127.39 103.75)
+		(end 126.89 104.25)
+		(width 1)
+		(layer "F.Cu")
+		(net "+6V")
+	)
+	(segment
 		(start 142.5 125.5)
 		(end 140.5 127.5)
@@
 	)
 	(segment
+		(start 134.25 103.75)
+		(end 127.39 103.75)
+		(width 1)
+		(layer "F.Cu")
+		(net "+6V")
+	)
+	(segment
+		(start 138.5 108)
+		(end 134.25 103.75)
+		(width 1)
+		(layer "F.Cu")
+		(net "+6V")
+	)
+	(segment
 		(start 157.5 108)
 		(end 160 110.5)
@@
 	)
 	(segment
-		(start 204.5 127.46)
-		(end 204.5 139)
+		(start 143.5 101.5)
+		(end 126.6 101.5)
 		(width 0.5)
 		(layer "B.Cu")
@@
 	)
 	(segment
-		(start 133.46 148.5)
-		(end 134.96 147)
+		(start 204.5 127.46)
+		(end 204.5 139)
 		(width 0.5)
 		(layer "B.Cu")
@@
 	)
 	(segment
-		(start 143.5 101.5)
-		(end 126.6 101.5)
+		(start 133.46 148.5)
+		(end 134.96 147)
 		(width 0.5)
 		(layer "B.Cu")
@@
 	)
 	(segment
-		(start 126.6 101.5)
-		(end 124.35 103.75)
+		(start 104.5 140.5)
+		(end 112.5 148.5)
 		(width 0.5)
 		(layer "B.Cu")
@@
 	)
 	(segment
-		(start 104.5 140.5)
-		(end 112.5 148.5)
+		(start 167 147)
+		(end 134.96 147)
 		(width 0.5)
 		(layer "B.Cu")
@@
 	)
 	(segment
-		(start 167 147)
-		(end 134.96 147)
+		(start 126.6 101.5)
+		(end 124.35 103.75)
 		(width 0.5)
 		(layer "B.Cu")
@@
 	)
 	(segment
+		(start 124.35 103.75)
+		(end 124.35 104.25)
+		(width 0.5)
+		(layer "B.Cu")
+		(net "+3V3")
+	)
+	(segment
 		(start 204.5 139)
 		(end 201 142.5)
@@
 	)
 	(segment
-		(start 125.52 110)
-		(end 161 110)
+		(start 119.27 104.25)
+		(end 125.02 110)
 		(width 0.3)
 		(layer "B.Cu")
@@
 	)
 	(segment
-		(start 119.27 103.75)
-		(end 125.52 110)
+		(start 125.02 110)
+		(end 161 110)
 		(width 0.3)
 		(layer "B.Cu")
@@
 	)
 	(segment
-		(start 123.98 111)
-		(end 174.5 111)
+		(start 116.73 104.25)
+		(end 123.48 111)
 		(width 0.3)
 		(layer "B.Cu")
@@
 	)
 	(segment
-		(start 116.73 103.75)
-		(end 123.98 111)
+		(start 123.48 111)
+		(end 174.5 111)
 		(width 0.3)
 		(layer "B.Cu")
@@
 	)
 	(segment
-		(start 123.852943 104.95)
-		(end 137.55 104.95)
-		(width 0.3)
-		(layer "B.Cu")
+		(start 116.44 102)
+		(end 137.5 102)
+		(width 0.2)
+		(layer "F.Cu")
 		(net "Net-(J6-Pin_1)")
 	)
 	(segment
-		(start 137.55 104.95)
+		(start 137.5 102)
 		(end 139 103.5)
-		(width 0.3)
-		(layer "B.Cu")
-		(net "Net-(J6-Pin_1)")
-	)
-	(segment
-		(start 123.15 103.252943)
-		(end 123.15 104.247057)
-		(width 0.3)
-		(layer "B.Cu")
-		(net "Net-(J6-Pin_1)")
-	)
-	(segment
-		(start 123.15 104.247057)
-		(end 123.852943 104.95)
-		(width 0.3)
-		(layer "B.Cu")
-		(net "Net-(J6-Pin_1)")
-	)
-	(segment
-		(start 114.19 103.75)
-		(end 115.39 102.55)
-		(width 0.3)
-		(layer "B.Cu")
-		(net "Net-(J6-Pin_1)")
-	)
-	(segment
-		(start 115.39 102.55)
-		(end 122.447057 102.55)
-		(width 0.3)
-		(layer "B.Cu")
+		(width 0.2)
+		(layer "F.Cu")
 		(net "Net-(J6-Pin_1)")
 	)
 	(segment
-		(start 122.447057 102.55)
-		(end 123.15 103.252943)
-		(width 0.3)
-		(layer "B.Cu")
+		(start 114.19 104.25)
+		(end 116.44 102)
+		(width 0.2)
+		(layer "F.Cu")
 		(net "Net-(J6-Pin_1)")
 	)
 	(segment
-		(start 111.65 103.75)
-		(end 114.4 101)
+		(start 111.65 104.25)
+		(end 111.65 103.75)
 		(width 0.3)
 		(layer "F.Cu")
@@
 	)
 	(segment
-		(start 201.24 111.3185)
-		(end 200.04 112.5185)
+		(start 111.65 103.75)
+		(end 114.4 101)
 		(width 0.3)
-		(layer "B.Cu")
-		(net "/pwm_B")
+		(layer "F.Cu")
+		(net "Net-(J6-Pin_6)")
 	)
 	(segment
-		(start 119.3815 112.5185)
+		(start 111.65 119.75)
 		(end 111.65 120.25)
 		(width 0.3)
@@
 	(segment
 		(start 200.04 112.5185)
-		(end 119.3815 112.5185)
+		(end 118.8815 112.5185)
 		(width 0.3)
 		(layer "B.Cu")
@@
 	)
 	(segment
-		(start 114.19 120.25)
+		(start 201.24 111.3185)
+		(end 200.04 112.5185)
+		(width 0.3)
+		(layer "B.Cu")
+		(net "/pwm_B")
+	)
+	(segment
+		(start 118.8815 112.5185)
+		(end 111.65 119.75)
+		(width 0.3)
+		(layer "B.Cu")
+		(net "/pwm_B")
+	)
+	(segment
+		(start 114.19 119.75)
 		(end 114.19 128.65)
 		(width 0.3)
@@
 	)
 	(segment
-		(start 116.73 120.25)
+		(start 116.73 119.75)
 		(end 116.73 128.65)
 		(width 0.3)
@@
 	)
 	(segment
-		(start 119.27 120.25)
+		(start 119.27 119.75)
 		(end 119.27 128.65)
 		(width 0.3)
@@
 	)
 	(segment
-		(start 121.81 120.25)
+		(start 121.81 119.75)
 		(end 121.81 128.65)
 		(width 0.3)
@@
 	)
 	(segment
-		(start 124.35 120.25)
+		(start 124.35 119.75)
 		(end 124.35 128.65)
 		(width 0.3)
@@
 	)
 	(segment
-		(start 131.14 124.5)
-		(end 126.89 120.25)
+		(start 201.24 113.8585)
+		(end 190.5985 124.5)
 		(width 0.3)
 		(layer "B.Cu")
@@
 	)
 	(segment
-		(start 201.24 113.8585)
-		(end 190.5985 124.5)
+		(start 190.5985 124.5)
+		(end 131.64 124.5)
 		(width 0.3)
 		(layer "B.Cu")
@@
 	)
 	(segment
-		(start 190.5985 124.5)
-		(end 131.14 124.5)
+		(start 131.64 124.5)
+		(end 126.89 119.75)
 		(width 0.3)
 		(layer "B.Cu")
@@
 		(polygon
 			(pts
-				(xy 134.5 136) (xy 137 135) (xy 138.5 142) (xy 136.5 143) (xy 134 138)
+				(xy 151.5 134) (xy 154 133) (xy 154 137) (xy 151 136)
 			)
 		)

Commit message: カルマンフィルタの実装
Routing:
- net GND: vias 0 -> 41
